File: WALLOPS_BLUE_GEN/WALLOPS.kicad_pcb (KiCad board)
At the start: 2 copper layers, 55 x 68 mm, 31 parts, among them J1 JST-PH 1x9 Connector - WALLOP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, Q1 AO3401A, U1 VL53L8CX 0 (0x20; Zwicky), U2 VL58L8CX 1 (0x2A; Aristotle), U3 VL53L8CX 3 (0x2C; Copernicus), U4 VL53L8CX 2 (0x2B; Brahe), U5 6DOF IMU (0x69; Sisko), U6 5V to 3.3V Converter

Commit message: Cleaned up WALLOPS PCB and added silkscreen
Parts:
- added G***: LOGO, LOGO, B.Cu at (187.8, 96.6)
- added G***: LOGO, LOGO, B.Cu at (207.7, 44.8)
