File: WALLOPS_REDEMPTION_ARC/WALLOPS_REDEMPTION_ARC.kicad_pcb (KiCad board)
At the start: 2 copper layers, 15.4 x 15.4 mm, 39 parts, among them J1 Power Connector, J2 I2C Connector, U1 PCA9306DC, U2 AP2112K-1.8, U3 5V to 3.3V Converter, U4 VL53L8CXV0GC/1

Commit message: Updated schematic
Parts:
- added C10: 100nF, Capacitor_SMD:C_0805_2012Metric_Pad1.18x1.45mm_HandSolder, F.Cu at (91.8, 95.8)
- added C11: 4.7μF, Capacitor_SMD:C_0805_2012Metric_Pad1.18x1.45mm_HandSolder, F.Cu at (91.8, 98.8)
- added C12: 100nF, Capacitor_SMD:C_0805_2012Metric_Pad1.18x1.45mm_HandSolder, F.Cu at (91.8, 101.8)
- added C13: 100nF, Capacitor_SMD:C_0805_2012Metric_Pad1.18x1.45mm_HandSolder, F.Cu at (91.8, 104.8)
- added C14: 4.7μF, Capacitor_SMD:C_0805_2012Metric_Pad1.18x1.45mm_HandSolder, F.Cu at (91.8, 107.8)
- added C15: 100nF, Capacitor_SMD:C_0805_2012Metric_Pad1.18x1.45mm_HandSolder, F.Cu at (91.8, 110.8)
- added C16: 100nF, Capacitor_SMD:C_0805_2012Metric_Pad1.18x1.45mm_HandSolder, F.Cu at (91.8, 113.8)
- added C17: 4.7μF, Capacitor_SMD:C_0805_2012Metric_Pad1.18x1.45mm_HandSolder, F.Cu at (91.8, 116.8)
- added C18: 100nF, Capacitor_SMD:C_0805_2012Metric_Pad1.18x1.45mm_HandSolder, F.Cu at (88.2, 65.0)
- added C19: 100nF, Capacitor_SMD:C_0805_2012Metric_Pad1.18x1.45mm_HandSolder, F.Cu at (88.2, 68.0)
- added C20: 100nF, Capacitor_SMD:C_0805_2012Metric_Pad1.18x1.45mm_HandSolder, F.Cu at (88.2, 71.0)
- added C4: 22μF, Capacitor_SMD:C_0805_2012Metric_Pad1.18x1.45mm_HandSolder, F.Cu at (88.2, 50.0)
- added C5: 100nF, Capacitor_SMD:C_0805_2012Metric_Pad1.18x1.45mm_HandSolder, F.Cu at (91.8, 92.8)
- added C6: 22μF, Capacitor_SMD:C_0805_2012Metric_Pad1.18x1.45mm_HandSolder, F.Cu at (88.2, 53.0)
- added C7: 4.7μF, Capacitor_SMD:C_0805_2012Metric_Pad1.18x1.45mm_HandSolder, F.Cu at (88.2, 56.0)
- added C8: 100nF, Capacitor_SMD:C_0805_2012Metric_Pad1.18x1.45mm_HandSolder, F.Cu at (88.2, 59.0)
- added C9: 100nF, Capacitor_SMD:C_0805_2012Metric_Pad1.18x1.45mm_HandSolder, F.Cu at (88.2, 62.0)
- added D10: GREEN_LED, LED_SMD:LED_0805_2012Metric_Pad1.15x1.40mm_HandSolder, F.Cu at (96.6, 95.8)
- added D11: RED_LED, LED_SMD:LED_0805_2012Metric_Pad1.15x1.40mm_HandSolder, F.Cu at (119.5, 56.1)
- added D12: PURPLE_LED, LED_SMD:LED_0805_2012Metric_Pad1.15x1.40mm_HandSolder, F.Cu at (96.6, 98.9)
- added D13: RED_LED, LED_SMD:LED_0805_2012Metric_Pad1.15x1.40mm_HandSolder, F.Cu at (119.5, 59.1)
- added D14: GREEN_LED, LED_SMD:LED_0805_2012Metric_Pad1.15x1.40mm_HandSolder, F.Cu at (96.6, 101.9)
- added D15: RED_LED, LED_SMD:LED_0805_2012Metric_Pad1.15x1.40mm_HandSolder, F.Cu at (119.5, 62.1)
- added D16: PURPLE_LED, LED_SMD:LED_0805_2012Metric_Pad1.15x1.40mm_HandSolder, F.Cu at (96.6, 104.9)
- added D17: RED_LED, LED_SMD:LED_0805_2012Metric_Pad1.15x1.40mm_HandSolder, F.Cu at (119.5, 65.2)
- added D18: GREEN_LED, LED_SMD:LED_0805_2012Metric_Pad1.15x1.40mm_HandSolder, F.Cu at (96.6, 108.0)
- added D7: RED_LED, LED_SMD:LED_0805_2012Metric_Pad1.15x1.40mm_HandSolder, F.Cu at (119.5, 50.0)
- added D8: PURPLE_LED, LED_SMD:LED_0805_2012Metric_Pad1.15x1.40mm_HandSolder, F.Cu at (96.6, 92.8)
- added D9: RED_LED, LED_SMD:LED_0805_2012Metric_Pad1.15x1.40mm_HandSolder, F.Cu at (119.5, 53.0)
- added R11: 22Ω, Resistor_SMD:R_0805_2012Metric_Pad1.20x1.40mm_HandSolder, F.Cu at (93.0, 68.8)
- added R12: 22Ω, Resistor_SMD:R_0805_2012Metric_Pad1.20x1.40mm_HandSolder, F.Cu at (93.0, 71.7)
- added R13: 47kΩ, Resistor_SMD:R_0805_2012Metric_Pad1.20x1.40mm_HandSolder, F.Cu at (93.0, 74.7)
- added R14: 47kΩ, Resistor_SMD:R_0805_2012Metric_Pad1.20x1.40mm_HandSolder, F.Cu at (93.0, 77.6)
- added R15: 47kΩ, Resistor_SMD:R_0805_2012Metric_Pad1.20x1.40mm_HandSolder, F.Cu at (93.0, 80.6)
- added R16: 22Ω, Resistor_SMD:R_0805_2012Metric_Pad1.20x1.40mm_HandSolder, F.Cu at (93.0, 83.5)
- added R17: 33Ω, Resistor_SMD:R_0805_2012Metric_Pad1.20x1.40mm_HandSolder, F.Cu at (101.4, 98.6)
- added R18: 47kΩ, Resistor_SMD:R_0805_2012Metric_Pad1.20x1.40mm_HandSolder, F.Cu at (97.8, 68.8)
- added R19: 22Ω, Resistor_SMD:R_0805_2012Metric_Pad1.20x1.40mm_HandSolder, F.Cu at (97.8, 71.7)
- added R20: 120 Ω, Resistor_SMD:R_0805_2012Metric_Pad1.20x1.40mm_HandSolder, F.Cu at (101.4, 101.6)
- added R21: 47kΩ, Resistor_SMD:R_0805_2012Metric_Pad1.20x1.40mm_HandSolder, F.Cu at (101.4, 104.5)
- added R22: 47kΩ, Resistor_SMD:R_0805_2012Metric_Pad1.20x1.40mm_HandSolder, F.Cu at (106.1, 92.7)
- added R23: 47kΩ, Resistor_SMD:R_0805_2012Metric_Pad1.20x1.40mm_HandSolder, F.Cu at (97.8, 74.7)
- added R24: 22Ω, Resistor_SMD:R_0805_2012Metric_Pad1.20x1.40mm_HandSolder, F.Cu at (97.8, 77.6)
- added R25: 33Ω, Resistor_SMD:R_0805_2012Metric_Pad1.20x1.40mm_HandSolder, F.Cu at (106.1, 95.7)
- added R26: 47kΩ, Resistor_SMD:R_0805_2012Metric_Pad1.20x1.40mm_HandSolder, F.Cu at (97.8, 80.6)
- added R27: 22Ω, Resistor_SMD:R_0805_2012Metric_Pad1.20x1.40mm_HandSolder, F.Cu at (97.8, 83.5)
- added R28: 120 Ω, Resistor_SMD:R_0805_2012Metric_Pad1.20x1.40mm_HandSolder, F.Cu at (106.1, 98.6)
- added R29: 47kΩ, Resistor_SMD:R_0805_2012Metric_Pad1.20x1.40mm_HandSolder, F.Cu at (106.1, 101.6)
- added R30: 47kΩ, Resistor_SMD:R_0805_2012Metric_Pad1.20x1.40mm_HandSolder, F.Cu at (106.1, 104.5)
- added R31: 47kΩ, Resistor_SMD:R_0805_2012Metric_Pad1.20x1.40mm_HandSolder, F.Cu at (102.5, 68.8)
- added R32: 22Ω, Resistor_SMD:R_0805_2012Metric_Pad1.20x1.40mm_HandSolder, F.Cu at (102.5, 71.7)
- added R33: 33Ω, Resistor_SMD:R_0805_2012Metric_Pad1.20x1.40mm_HandSolder, F.Cu at (110.9, 92.7)
- added R34: 47kΩ, Resistor_SMD:R_0805_2012Metric_Pad1.20x1.40mm_HandSolder, F.Cu at (102.5, 74.7)
- added R35: 22Ω, Resistor_SMD:R_0805_2012Metric_Pad1.20x1.40mm_HandSolder, F.Cu at (102.5, 77.6)
- added R36: 120 Ω, Resistor_SMD:R_0805_2012Metric_Pad1.20x1.40mm_HandSolder, F.Cu at (110.9, 95.7)
- added R37: 47kΩ, Resistor_SMD:R_0805_2012Metric_Pad1.20x1.40mm_HandSolder, F.Cu at (110.9, 98.6)
- added R38: 47kΩ, Resistor_SMD:R_0805_2012Metric_Pad1.20x1.40mm_HandSolder, F.Cu at (110.9, 101.6)
- added TP13: L2_TP, TestPoint:TestPoint_Pad_D1.0mm, F.Cu at (108.6, 113.6)
- added TP16: L1_TP, TestPoint:TestPoint_Pad_D1.0mm, F.Cu at (111.7, 113.6)
- added TP19: L3_TP, TestPoint:TestPoint_Pad_D1.0mm, F.Cu at (114.7, 113.6)
- added U10: ISM330DHCX, RockSat:ISM330DHCX, F.Cu at (104.3, 56.7)
- added U5: Schottky Diode, Package_TO_SOT_SMD:TO-277B, F.Cu at (107.7, 71.7)
- added U6: SN74LVC125ADR, RockSat:SOIC127P600X175-14N, F.Cu at (124.1, 82.4)
- added U7: VL53L8CXV0GC/1, RockSat:vl53l8cx_smd, F.Cu at (103.1, 108.4)
- added U8: VL53L8CXV0GC/1, RockSat:vl53l8cx_smd, F.Cu at (103.1, 113.1)
- added U9: VL53L8CXV0GC/1, RockSat:vl53l8cx_smd, F.Cu at (103.1, 117.8)
- D4, D5: value WHITE_LED -> RED_LED
- J1: footprint Connector_JST:JST_PH_S4B-PH-K_1x04_P2.00mm_Horizontal -> Connector_JST:JST_PH_S7B-PH-K_1x07_P2.00mm_Horizontal
- R10: value ??? Ω -> 120 Ω
- R8, R9: value ??? Ω -> 4.7kΩ
- U1: value PCA9306DC -> TCA9517DR; footprint Package_SO:VSSOP-8_2.3x2mm_P0.5mm -> RockSat:SOIC127P599X175-8N
- moved R8 45.3 mm to (101.4, 92.7)
- moved R9 45.3 mm to (101.4, 95.7)
Connections:
- R8 pad 1: /1V8 -> /3V3
- R8 pad 2: Net-(D4-A) -> /SDA
- R9 pad 1: /1V8 -> /3V3
- R9 pad 2: Net-(D5-A) -> /SCL
- U1 pad 1: GND -> /1V8
- U1 pad 2: /3V3 -> /SCL
- U1 pad 3: /SCL -> /SDA
- U1 pad 4: /SDA -> GND
- U1 pad 5: /SCL -> /3V3
- U1 pad 7: /1V8 -> /SCL
- U1 pad 8: unconnected-(U1-EN-Pad8) -> /3V3
- U2 pad 3: unconnected-(U2-EN-Pad3) -> /3V3
- U4 pad A1: unconnected-(U4-INT-PadA1) -> Net-(U4-INT)
- U4 pad A4: /SCL -> /SDA
- U4 pad A5: /SDA -> /SCL
- U4 pad B1: unconnected-(U4-SYNC-PadB1) -> Net-(U4-SYNC)
Routing:
- added copper zone on B.Cu, net (none)
Other:
- board size 15.4 x 15.4 mm -> 25.4 x 17.8 mm

Commit message: Added base PCB dimensions
Parts:
- added G***: LOGO, LOGO, F.Cu at (186.3, 149.9)
- moved C1 117.7 mm to (22.8, 130.2)
- moved C10 117.7 mm to (-25.5, 105.4)
- moved C11 117.7 mm to (-25.5, 108.4)
- moved C12 117.7 mm to (-25.5, 111.4)
- moved C13 117.7 mm to (-25.5, 114.4)
- moved C14 117.7 mm to (-25.5, 117.5)
- moved C15 117.7 mm to (-25.5, 120.5)
- moved C16 117.7 mm to (-25.5, 123.5)
- moved C17 117.7 mm to (-25.5, 126.5)
- moved C18 117.7 mm to (-29.1, 74.7)
- moved C19 117.7 mm to (-29.1, 77.7)
- moved C2 117.7 mm to (22.8, 133.2)
- moved C20 117.7 mm to (-29.1, 80.7)
- moved C3 117.7 mm to (22.8, 136.2)
- moved C4 117.7 mm to (-29.1, 59.6)
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Routing:
- net /3V3: track 35.5 -> 0.00 mm
- net /5V: track 23.2 -> 0.00 mm
- net GND: track 6.70 -> 0.00 mm
Other:
- board size 25.4 x 17.8 mm -> 57 x 72.1 mm
- board text added: "Made by Mark, Tatiana, Laura, and Aidan"
- board text added: "Wide Angle LiDAR Laser Operating in Space"
- board text added: "w a l l o p s"

Commit message: Added passives for power side of PCB
Parts:
- removed C8, C9: 100nF, Capacitor_SMD:C_0805_2012Metric_Pad1.18x1.45mm_HandSolder
- removed TP3: SCH_TP, TestPoint:TestPoint_Pad_D1.0mm
- C4, TP2, U5: moved to B.Cu
- TP7: value 3SD_TP -> SCL_TP
- TP8: value 3SC_TP -> SD_TP
- moved D18 182.3 mm to (161.1, 130.9), turned to 180 degrees
- moved D16 181.9 mm to (161.1, 120.2), turned to 180 degrees
- moved D14 179.0 mm to (158.3, 113.1), turned to 180 degrees
- moved D12 178.7 mm to (158.0, 107.5), turned to 180 degrees
- moved R32 177.3 mm to (157.3, 123.9)
- moved R35 176.8 mm to (157.4, 127.6)
- moved R24 175.3 mm to (154.3, 109.8)
- moved R27 174.0 mm to (154.1, 104.2)
- moved D17 167.5 mm to (161.1, 127.6), turned to 180 degrees
- moved D15 167.2 mm to (161.1, 123.9), turned to 180 degrees
- moved R36 165.8 mm to (157.4, 130.9), turned to 180 degrees
- moved R28 165.8 mm to (154.5, 113.1), turned to 180 degrees
- moved R25 165.5 mm to (154.3, 107.5)
- moved R33 164.8 mm to (157.4, 120.2), turned to 180 degrees
- moved C17 164.4 mm to (138.8, 120.9)
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Connections:
- J2 pad 2: /SCL -> /SDA
- J2 pad 4: /SDA -> /SCL
- TP7 pad 1: /SDA -> /SCL
- TP8 pad 1: /SCL -> /SDA
Routing:
- net /3V3: track 0.00 -> 78.6 mm, vias 0 -> 1
- net /LPn_3: track 0.00 -> 54.6 mm
- net /LPn_2: track 0.00 -> 53.6 mm
- net /SDA: track 0.00 -> 46.7 mm
- net /SCL: track 0.00 -> 46.5 mm
- net /SCAN: track 0.00 -> 44.8 mm
- net /LPn_1: track 0.00 -> 41.7 mm
- net /5V: track 0.00 -> 39.2 mm, vias 0 -> 1
- net /LPn_0: track 0.00 -> 38.7 mm
- net /1V8: track 0.00 -> 29.6 mm
- net GND: track 0.00 -> 26.4 mm, vias 1 -> 13
- net Net-(D2-A): track 0.00 -> 1.82 mm
- net Net-(D1-A): track 0.00 -> 1.80 mm
- added copper zone on B.Cu, net GND
- removed copper zone on B.Cu, net (none)
Other:
- board size 57 x 72.1 mm -> 57.1 x 72.6 mm
- board text added: "22μF"
- board text added: "LPn1"
- board text added: "LPn2"
- board text added: "LPn3"

Commit message: Updated Wallops Redemption ARC
Parts:
- removed D10, D14, D18, D6: GREEN_LED, LED_SMD:LED_0805_2012Metric_Pad1.15x1.40mm_HandSolder
- removed D11, D13, D15, D17, D4, D5, D7, D9: RED_LED, LED_SMD:LED_0805_2012Metric_Pad1.15x1.40mm_HandSolder
- removed R10, R20, R28, R36: 120 Ω, Resistor_SMD:R_0805_2012Metric_Pad1.20x1.40mm_HandSolder
- removed R11, R12, R16, R19, R24, R27, R32, R35: 22Ω, Resistor_SMD:R_0805_2012Metric_Pad1.20x1.40mm_HandSolder
- removed TP10: 1SC_TP, TestPoint:TestPoint_Pad_D1.0mm
- removed TP2: 5V_TP, TestPoint:TestPoint_Pad_D1.0mm
- removed TP9: 1SD_TP, TestPoint:TestPoint_Pad_D1.0mm
- removed U10: ISM330DHCX, RockSat:ISM330DHCX
- added G***: LOGO, LOGO, F.Cu at (142.4, 110.7)
- added G***: LOGO, LOGO, F.Cu at (118.0, 95.2)
- added G***: LOGO, LOGO, F.Cu at (92.0, 79.5)
- added G***: LOGO, LOGO, F.Cu at (96.0, 116.3)
- added G***: LOGO, LOGO, F.Cu at (93.7, 105.8)
- added G***: LOGO, LOGO, B.Cu at (119.2, 86.5)
- C4, U5: moved to F.Cu
- C6: moved to B.Cu
- TP1: value GND_TP -> 5V_TP
- TP8: value SD_TP -> SDA_TP
- moved G*** 46.7 mm to (134.6, 89.9)
- moved J2 44.1 mm to (101.1, 68.0), turned to 180 degrees
- moved TP7 41.6 mm to (95.2, 74.7)
- moved R9 41.6 mm to (93.2, 71.8), turned to 90 degrees
- moved D8 39.8 mm to (115.6, 129.5), turned to 180 degrees
- moved TP19 39.7 mm to (113.2, 84.2)
- moved R8 39.4 mm to (101.0, 71.8)
- moved D3 38.5 mm to (115.0, 110.5), turned to 180 degrees
- moved TP8 38.2 mm to (99.1, 74.6)
- moved TP13 34.6 mm to (109.3, 84.2)
- moved R17 32.4 mm to (111.8, 129.5), turned to 180 degrees
- moved C19 31.7 mm to (93.6, 88.4), turned to 90 degrees
- moved U1 31.3 mm to (97.1, 81.9), turned to 90 degrees
- moved R5 31.1 mm to (111.3, 110.5), turned to 180 degrees
- moved C20 26.5 mm to (106.2, 79.9), turned to 90 degrees
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Connections:
- J1 pad 2: /5V -> /5Vin
- J1 pad 4: /LPn_0 -> /LPn_0_3V3
- J1 pad 5: /LPn_1 -> /LPn_1_3V3
- J1 pad 6: /LPn_2 -> /LPn_2_3V3
- J1 pad 7: /LPn_3 -> /LPn_3_3V3
- J2 pad 2: /SDA -> /SDA_3V3
- J2 pad 4: /SCL -> /SCL_3V3
- R8 pad 2: /SDA -> /SDA_3V3
- R9 pad 2: /SCL -> /SCL_3V3
- TP1 pad 1: GND -> /5V
- TP7 pad 1: /SCL -> /SCL_3V3
- TP8 pad 1: /SDA -> /SDA_3V3
- U1 pad 6: /SDA -> /SDA_3V3
- U1 pad 7: /SCL -> /SCL_3V3
- U5 pad 1: /5V -> /5Vin
- U5 pad 2: /5V -> /5Vin
- U6 pad 12: /LPn_3 -> /LPn_3_3V3
- U6 pad 2: /LPn_0 -> /LPn_0_3V3
- U6 pad 5: /LPn_1 -> /LPn_1_3V3
- U6 pad 9: /LPn_2 -> /LPn_2_3V3
Routing:
- net /1V8: track 29.6 -> 296.5 mm, vias 0 -> 15
- net /3V3: track 78.6 -> 232.4 mm, vias 1 -> 8
- net /SDA: track 46.7 -> 179.6 mm
- net /SCL: track 46.5 -> 160.9 mm
- net GND: track 26.4 -> 83.9 mm, vias 13 -> 82
- net /SCAN: track 44.8 -> 4.11 mm
- net /LPn_3: track 54.6 -> 84.3 mm, vias 0 -> 3
- net /LPn_2_3V3: track 0.00 -> 24.1 mm
- net /5V: track 39.2 -> 21.1 mm, vias 1 -> 0
- net /LPn_3_3V3: track 0.00 -> 17.3 mm
- net /LPn_1: track 41.7 -> 58.3 mm, vias 0 -> 3
- net /SDA_3V3: track 0.00 -> 14.2 mm
- net /SCL_3V3: track 0.00 -> 14.1 mm
- net /LPn_0: track 38.7 -> 48.0 mm, vias 0 -> 2
- net /LPn_1_3V3: track 0.00 -> 8.04 mm
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Other:
- outline, holes or cut-outs redrawn
- board text added: "*"
- board text added: "100nF"
- board text added: "1V8"
- board text added: "2kΩ"
- board text added: "33Ω"
- board text added: "4.7kΩ"
- board text added: "4.7μF"
- board text added: "47kΩ"
- board text added: "ARISTOTLE (0x2A)"
- board text added: "BRAHE (0x2B)"
- board text added: "COPERNICUS (0x2C)"
- board text added: "D24V22F3"
- board text added: "I2C"
- board text added: "LPn 0"
- board text added: "LPn 1"
- board text added: "LPn 2"
- board text added: "LPn 3"
- board text added: "Power"
- board text added: "Purple"
- board text added: "ZWICKY (0x20)"
