File: WALLOPS_REDEMPTION_ARC/WALLOPS_REDEMPTION_ARC.kicad_sch (KiCad schematic)
At the start: 49 parts, among them J1 Power Connector, J2 I2C Connector, U1 TCA9517DR, U2 AP2112K-1.8, U3 5V to 3.3V Converter, U4 VL53L8CXV0GC/1, U5 Schottky Diode, U6 SN74LVC125ADR

Commit message: Added current schematic for WALLOPS
Parts:
- removed C5: 1μF, symbol Device:C
- C4: value ? F -> 100μF
Connections:
- net GND: now also U6.7 (GND)
- net LPn_0: now also U6.3 (1Y)
Other:
- note added: "Use voltage divider instead of level shifter?"
- note removed: "!!!DOES LPN NEED LEVEL SHIFTER????"
Changed lines of the file:
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@@
 		)
 	)
-	(text "!!!DOES LPN NEED LEVEL SHIFTER????"
+	(text "Use voltage divider instead of level shifter?"
 		(exclude_from_sim no)
-		(at 139.446 115.824 0)
+		(at 236.982 78.486 0)
 		(effects
 			(font
@@
 	)
 	(junction
-		(at 143.51 52.07)
-		(diameter 0)
-		(color 0 0 0 0)
-	)
-	(junction
 		(at 72.39 109.22)
 		(diameter 0)
@@
 	(wire
 		(pts
-			(xy 143.51 52.07) (xy 144.78 52.07)
-		)
-		(stroke
-			(width 0)
-			(type default)
-		)
-	)
-	(wire
-		(pts
 			(xy 162.56 52.07) (xy 166.37 52.07)
 		)
@@
 	(wire
 		(pts
-			(xy 143.51 52.07) (xy 143.51 59.69)
-		)
-		(stroke
-			(width 0)
-			(type default)
-		)
-	)
-	(wire
-		(pts
 			(xy 72.39 123.19) (xy 72.39 109.22)
 		)
@@
 	(wire
 		(pts
-			(xy 46.99 44.45) (xy 46.99 58.42)
-		)
-		(stroke
-			(width 0)
-			(type default)
-		)
-	)
-	(wire
-		(pts
 			(xy 100.33 127) (xy 104.14 127)
 		)
@@
 	(wire
 		(pts
+			(xy 46.99 44.45) (xy 46.99 58.42)
+		)
+		(stroke
+			(width 0)
+			(type default)
+		)
+	)
+	(wire
+		(pts
 			(xy 101.6 63.5) (xy 104.14 63.5)
 		)
@@
 	(wire
 		(pts
-			(xy 143.51 67.31) (xy 143.51 71.12)
-		)
-		(stroke
-			(width 0)
-			(type default)
-		)
-	)
-	(wire
-		(pts
 			(xy 46.99 58.42) (xy 58.42 58.42)
 		)
@@
 	(wire
 		(pts
+			(xy 166.37 82.55) (xy 179.07 82.55)
+		)
+		(stroke
+			(width 0)
+			(type default)
+		)
+	)
+	(wire
+		(pts
 			(xy 137.16 54.61) (xy 139.7 54.61)
 		)
@@
 	(wire
 		(pts
-			(xy 139.7 52.07) (xy 143.51 52.07)
+			(xy 139.7 52.07) (xy 144.78 52.07)
 		)
 		(stroke
@@
 	(wire
 		(pts
-			(xy 85.09 90.17) (xy 176.53 90.17)
+			(xy 85.09 90.17) (xy 204.47 90.17)
 		)
 		(stroke
@@
 	(wire
 		(pts
+			(xy 204.47 82.55) (xy 204.47 90.17)
+		)
+		(stroke
+			(width 0)
+			(type default)
+		)
+	)
+	(wire
+		(pts
 			(xy 130.81 54.61) (xy 132.08 54.61)
 		)
@@
 	)
 	(label "SDA"
-		(at 46.99 44.45 90)
+		(at 46.99 50.8 90)
 		(effects
 			(font
@@
 			)
 		)
-		(property "Value" "? F"
+		(property "Value" "100μF"
 			(at 101.6 57.15 90)
 			(effects
@@
 	(symbol
 		(lib_id "power:GND")
+		(at 166.37 82.55 270)
+		(unit 1)
+		(exclude_from_sim no)
+		(in_bom yes)
+		(on_board yes)
+		(dnp no)
+		(property "Reference" "#PWR028"
+			(at 160.02 82.55 0)
+			(effects
+				(font
+					(size 1.27 1.27)
+				)
+				(hide yes)
+			)
+		)
+		(property "Value" "GND"
+			(at 162.306 82.55 0)
+			(effects
+				(font
+					(size 1.27 1.27)
+				)
+			)
+		)
+		(property "Footprint" ""
+			(at 166.37 82.55 0)
+			(effects
+				(font
+					(size 1.27 1.27)
+				)
+				(hide yes)
+			)
+		)
+		(property "Datasheet" ""
+			(at 166.37 82.55 0)
+			(effects
+				(font
+					(size 1.27 1.27)
+				)
+				(hide yes)
+			)
+		)
+		(property "Description" "Power symbol creates a global label with name \"GND\" , ground"
+			(at 166.37 82.55 0)
+			(effects
+				(font
+					(size 1.27 1.27)
+				)
+				(hide yes)
+			)
+		)
+		(pin "1"
+		)
+		(instances
+			(project "WALLOPS_REDEMPTION_ARC"
+				(path "/e70a348f-eac5-4047-8b06-1092c268c28a"
+					(reference "#PWR028")
+					(unit 1)
+				)
+			)
+		)
+	)
+	(symbol
+		(lib_id "power:GND")
 		(at 92.71 69.85 0)
 		(unit 1)
@@
 	)
 	(symbol
-		(lib_id "Device:C")
-		(at 143.51 63.5 0)
-		(unit 1)
-		(exclude_from_sim no)
-		(in_bom yes)
-		(on_board yes)
-		(dnp no)
-		(property "Reference" "C5"
-			(at 146.304 61.976 0)
-			(effects
-				(font
-					(size 1.27 1.27)
-				)
-				(justify left)
-			)
-		)
-		(property "Value" "1μF"
-			(at 146.304 64.516 0)
-			(effects
-				(font
-					(size 1.27 1.27)
-				)
-				(justify left)
-			)
-		)
-		(property "Footprint" ""
-			(at 144.4752 67.31 0)
-			(effects
-				(font
-					(size 1.27 1.27)
-				)
-				(hide yes)
-			)
-		)
-		(property "Datasheet" "~"
-			(at 143.51 63.5 0)
-			(effects
-				(font
-					(size 1.27 1.27)
-				)
-				(hide yes)
-			)
-		)
-		(property "Description" "Unpolarized capacitor"
-			(at 143.51 63.5 0)
-			(effects
-				(font
-					(size 1.27 1.27)
-				)
-				(hide yes)
-			)
-		)
-		(pin "1"
-		)
-		(pin "2"
-		)
-		(instances
-			(project "WALLOPS_REDEMPTION_ARC"
-				(path "/e70a348f-eac5-4047-8b06-1092c268c28a"
-					(reference "C5")
-					(unit 1)
-				)
-			)
-		)
-	)
-	(symbol
 		(lib_id "Device:LED")
 		(at 96.52 100.33 270)
@@
 					(unit 1)
 				)
-			)
-		)
-	)
-	(symbol
-		(lib_id "power:GND")
-		(at 143.51 71.12 0)
-		(unit 1)
-		(exclude_from_sim no)
-		(in_bom yes)
-		(on_board yes)
-		(dnp no)
-		(property "Reference" "#PWR023"
-			(at 143.51 77.47 0)
-			(effects
-				(font
-					(size 1.27 1.27)
-				)
-				(hide yes)
-			)
-		)
-		(property "Value" "GND"
-			(at 143.51 75.184 0)
-			(effects
-				(font
-					(size 1.27 1.27)
-				)
-			)
-		)
-		(property "Footprint" ""
-			(at 143.51 71.12 0)
-			(effects
-				(font
-					(size 1.27 1.27)
-				)
-				(hide yes)
-			)
-		)
-		(property "Datasheet" ""
-			(at 143.51 71.12 0)
-			(effects
-				(font
-					(size 1.27 1.27)
-				)
-				(hide yes)
-			)
-		)
-		(property "Description" "Power symbol creates a global label with name \"GND\" , ground"
-			(at 143.51 71.12 0)
-			(effects
-				(font
-					(size 1.27 1.27)
-				)
-				(hide yes)
-			)
-		)
-		(pin "1"
-		)
-		(instances
-			(project "WALLOPS_REDEMPTION_ARC"
-				(path "/e70a348f-eac5-4047-8b06-1092c268c28a"
-					(reference "#PWR023")
-					(unit 1)
-				)

Commit message: Updated schematic
Parts:
- added C10, C12, C13, C15, C16, C18, C19, C20, C5: 100nF, Capacitor_SMD:C_0805_2012Metric_Pad1.18x1.45mm_HandSolder, symbol Device:C
- added C11, C14, C17: 4.7μF, Capacitor_SMD:C_0805_2012Metric_Pad1.18x1.45mm_HandSolder, symbol Device:C
- added D10, D14, D18: GREEN_LED, LED_SMD:LED_0805_2012Metric_Pad1.15x1.40mm_HandSolder, symbol Device:LED
- added D11, D13, D15, D17, D7, D9: RED_LED, LED_SMD:LED_0805_2012Metric_Pad1.15x1.40mm_HandSolder, symbol Device:LED
- added D12, D16, D8: PURPLE_LED, LED_SMD:LED_0805_2012Metric_Pad1.15x1.40mm_HandSolder, symbol Device:LED
- added R15, R18, R21, R22, R23, R26, R29, R30, R31, R34, R37, R38: 47kΩ, Resistor_SMD:R_0805_2012Metric_Pad1.20x1.40mm_HandSolder, symbol Device:R_US
- added R16, R19, R24, R27, R32, R35: 22Ω, Resistor_SMD:R_0805_2012Metric_Pad1.20x1.40mm_HandSolder, symbol Device:R_US
- added R17, R25, R33: 33Ω, Resistor_SMD:R_0805_2012Metric_Pad1.20x1.40mm_HandSolder, symbol Device:R_US
- added R20, R28, R36: 120 Ω, Resistor_SMD:R_0805_2012Metric_Pad1.20x1.40mm_HandSolder, symbol Device:R_US
- added R8, R9: 4.7kΩ, Resistor_SMD:R_0805_2012Metric_Pad1.20x1.40mm_HandSolder, symbol Device:R_US
- added TP13: L2_TP, TestPoint:TestPoint_Pad_D1.0mm, symbol Connector:TestPoint
- added TP16: L1_TP, TestPoint:TestPoint_Pad_D1.0mm, symbol Connector:TestPoint
- added TP19: L3_TP, TestPoint:TestPoint_Pad_D1.0mm, symbol Connector:TestPoint
- added U10: ISM330DHCX, RockSat:ISM330DHCX, symbol RockSat:ISM330DHCX
- added U7, U8, U9: VL53L8CXV0GC/1, RockSat:vl53l8cx_smd, symbol RockSat:VL53L8CXV0GC_SMD
- C4: value 100μF -> 22μF; footprint (none) -> Capacitor_SMD:C_0805_2012Metric_Pad1.18x1.45mm_HandSolder
- C6: value 47μF -> 22μF; footprint (none) -> Capacitor_SMD:C_0805_2012Metric_Pad1.18x1.45mm_HandSolder
- C7: value 22μF -> 4.7μF; footprint (none) -> Capacitor_SMD:C_0805_2012Metric_Pad1.18x1.45mm_HandSolder
- C8, C9: value 0.1μF -> 100nF; footprint (none) -> Capacitor_SMD:C_0805_2012Metric_Pad1.18x1.45mm_HandSolder
- D4, D5: footprint (none) -> LED_SMD:LED_0805_2012Metric_Pad1.15x1.40mm_HandSolder
- J1: footprint Connector_JST:JST_PH_S4B-PH-K_1x04_P2.00mm_Horizontal -> Connector_JST:JST_PH_S7B-PH-K_1x07_P2.00mm_Horizontal
- R11, R12, R13, R14: footprint (none) -> Resistor_SMD:R_0805_2012Metric_Pad1.20x1.40mm_HandSolder
- U5: footprint (none) -> Package_TO_SOT_SMD:TO-277B
Connections:
- net 1V8: now also U1.1 (VCCA), U6.14 (VCC), C10.1, C12.1, C13.1, C15.1, C16.1, C18.1, C19.2, C5.1, R15.1, R16.1, R18.1, R19.1, R23.1, R24.1, R26.1, R27.1, R31.1, R32.1, R34.1, R35.1, U7.A3 (IOVDD), U7.B7 (CORE_1V8), U8.A3 (IOVDD), U8.B7 (CORE_1V8), U9.A3 (IOVDD), U9.B7 (CORE_1V8); no longer U1.8 (VCCB)
- net 3V3: now also U1.5 (EN), U1.8 (VCCB), U2.3 (EN), C11.2, C14.2, C17.2, C20.2, R20.2, R28.2, R36.2, R8.1, R9.1, U10.1 (VIN), U7.C4 (AVDD), U8.C4 (AVDD), U9.C4 (AVDD); no longer U1.1 (VCCA)
- net GND: now also U6.1 (1~OE), U6.10 (3~OE), U6.13 (4~OE), U6.4 (2~OE), C10.2, C11.1, C12.2, C13.2, C14.1, C15.2, C16.2, C17.1, C18.2, C19.1, C20.1, C5.2, D10.1 (K), D11.1 (K), D12.1 (K), D13.1 (K), D14.1 (K), D15.1 (K), D16.1 (K), D17.1 (K), D18.1 (K), D7.1 (K), D8.1 (K), D9.1 (K), R21.2, R22.2, R29.2, R30.2, R37.2, R38.2, U10.3 (GND), U7.A6 (RSVD1), U7.A7 (RSVD2), U7.B4 (THERMALPAD), U7.C3 (GND), U7.C6 (RSVD3), U7.C7 (GROUND), U8.A6 (RSVD1), U8.A7 (RSVD2), U8.B4 (THERMALPAD), U8.C3 (GND), U8.C6 (RSVD3), U8.C7 (GROUND), U9.A6 (RSVD1), U9.A7 (RSVD2), U9.B4 (THERMALPAD), U9.C3 (GND), U9.C6 (RSVD3), U9.C7 (GROUND)
- net LPn_0: now also U6.2 (1A)
- net LPn_1: now also U6.5 (2A), U6.6 (2Y), R25.2, TP16.1, U8.A2 (LPN)
- net LPn_2: now also U6.8 (3Y), U6.9 (3A), R17.2, TP13.1, U7.A2 (LPN)
- net LPn_3: now also U6.11 (4Y), U6.12 (4A), R33.2, TP19.1, U9.A2 (LPN)
- net SCL: now also U4.A5 (SCL/MCLK), R9.2, U10.4 (SCL), U7.A5 (SCL/MCLK), U8.A5 (SCL/MCLK), U9.A5 (SCL/MCLK); no longer U4.A4 (SDA/MOSI)
- net SDA: now also U4.A4 (SDA/MOSI), R8.2, U10.5 (SDA), U7.A4 (SDA/MOSI), U8.A4 (SDA/MOSI), U9.A4 (SDA/MOSI); no longer U4.A5 (SCL/MCLK)
- new net: R22.1, U7.C2 (NCS)
- new net: D7.2 (A), R16.2
- new net: D17.2 (A), R35.2
- new net: R31.2, U9.B1 (SYNC)
- new net: R26.2, U8.A1 (INT)
- new net: R34.2, U9.A1 (INT)
- new net: D18.2 (A), R36.1
- new net: D12.2 (A), R25.1
- new net: R29.1, U8.C1 (SPI_I2C_N)
- new net: D13.2 (A), R27.2
- new net: D10.2 (A), R20.1
- new net: R38.1, U9.C2 (NCS)
- new net: D15.2 (A), R32.2
- new net: R15.2, U7.B1 (SYNC)
- new net: R21.1, U7.C1 (SPI_I2C_N)
- new net: D8.2 (A), R17.1
- new net: D14.2 (A), R28.1
- new net: D16.2 (A), R33.1
- new net: R23.2, U8.B1 (SYNC)
- new net: D9.2 (A), R19.2
- new net: R18.2, U7.A1 (INT)
- new net: R37.1, U9.C1 (SPI_I2C_N)
- new net: D11.2 (A), R24.2
- new net: R30.1, U8.C2 (NCS)
- no-connect marks 6 -> 12
Other:
- note added: "Aristotle (0x2A)"
- note added: "Brahe (0x2B)"
- note added: "Copernicus (0x2C)"
- note added: "Level Shifter (Unidirectional; LPn)"
- note removed: "Use voltage divider instead of level shifter?"
- note removed: "^ THESE ARE THE 1V8 I2C PULL UPS"
- moved on the sheet: C1, C2, C3, C4, C6, C7, C8, C9, D1, D2, D3, D4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

Commit message: Added passives for power side of PCB
Parts:
- removed C8, C9: 100nF, Capacitor_SMD:C_0805_2012Metric_Pad1.18x1.45mm_HandSolder, symbol Device:C
- removed TP3: SCH_TP, TestPoint:TestPoint_Pad_D1.0mm, symbol Connector:TestPoint
- TP7: value 3SD_TP -> SCL_TP
- TP8: value 3SC_TP -> SD_TP
Connections:
- net SCL: now also J2.4 (Pin_4), TP7.1; no longer J2.2 (Pin_2), TP8.1
- net SDA: now also J2.2 (Pin_2), TP8.1; no longer J2.4 (Pin_4), TP7.1
Other:
- note removed: "Decoupling Capacitors"
- moved on the sheet: R8, TP7

Commit message: Updated Wallops Redemption ARC
Parts:
- removed D10, D14, D18, D6: GREEN_LED, LED_SMD:LED_0805_2012Metric_Pad1.15x1.40mm_HandSolder, symbol Device:LED
- removed D11, D13, D15, D17, D4, D5, D7, D9: RED_LED, LED_SMD:LED_0805_2012Metric_Pad1.15x1.40mm_HandSolder, symbol Device:LED
- removed R10, R20, R28, R36: 120 Ω, Resistor_SMD:R_0805_2012Metric_Pad1.20x1.40mm_HandSolder, symbol Device:R_US
- removed R11, R12, R16, R19, R24, R27, R32, R35: 22Ω, Resistor_SMD:R_0805_2012Metric_Pad1.20x1.40mm_HandSolder, symbol Device:R_US
- removed TP10: 1SC_TP, TestPoint:TestPoint_Pad_D1.0mm, symbol Connector:TestPoint
- removed TP2: 5V_TP, TestPoint:TestPoint_Pad_D1.0mm, symbol Connector:TestPoint
- removed TP9: 1SD_TP, TestPoint:TestPoint_Pad_D1.0mm, symbol Connector:TestPoint
- removed U10: ISM330DHCX, RockSat:ISM330DHCX, symbol RockSat:ISM330DHCX
- TP1: value GND_TP -> 5V_TP
- TP8: value SD_TP -> SDA_TP
Connections:
- net 5V: now also TP1.1; no longer J1.2 (Pin_2), U5.1 (VIN), U5.2 (VIN)
- net GND: no longer TP1.1
- net LPn_0: no longer J1.4 (Pin_4), U6.2 (1A)
- net LPn_1: no longer J1.5 (Pin_5), U6.5 (2A)
- net LPn_2: no longer J1.6 (Pin_6), U6.9 (3A)
- net LPn_3: no longer J1.7 (Pin_7), U6.12 (4A)
- net SCL: no longer J2.4 (Pin_4), R9.2, TP7.1, U1.7 (SCLB)
- net SDA: no longer J2.2 (Pin_2), R8.2, TP8.1, U1.6 (SDAB)
- new net 5Vin: J1.2 (Pin_2), U5.1 (VIN), U5.2 (VIN)
- new net LPn_0_3V3: J1.4 (Pin_4), U6.2 (1A)
- new net LPn_1_3V3: J1.5 (Pin_5), U6.5 (2A)
- new net LPn_2_3V3: J1.6 (Pin_6), U6.9 (3A)
- new net LPn_3_3V3: J1.7 (Pin_7), U6.12 (4A)
- new net SCL_3V3: J2.4 (Pin_4), R9.2, TP7.1, U1.7 (SCLB)
- new net SDA_3V3: J2.2 (Pin_2), R8.2, TP8.1, U1.6 (SDAB)
- no-connect marks 12 -> 7
Other:
- note removed: "Green LED turns on when 3.3V is successfully delivered through the line."
- note removed: "RED LEDs indicate that the VL53L8CX is successfully receiving 1V8."
- moved on the sheet: C1, C10, C11, C12, C13, C14, C15, C16, C17, C18, C19, C2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
